File: kicad/iot_power/iot_power.kicad_pcb (KiCad board)
At the start: 2 copper layers, 60 x 100 mm, 16 parts, among them J1 POWER_SOURCE, J2 RELAY, J3 OLED, J4 PZEM004T, U1 L7805CV

Commit message: nov 25
Parts:
- removed 11: ESP32-DevKitC, Espressif:ESP32-Nodemcu-india
- removed kibuzzard-67C6BA96: G***, kibuzzard-67C6BA96
- added D4: 1N4148, Diode_THT:D_DO-35_SOD27_P7.62mm_Horizontal, F.Cu at (30.1, 82.3)
- added D5: LED, LED_THT:LED_D3.0mm, F.Cu at (37.6, 86.0)
- added K1: G5LE-1, Relay_THT:Relay_SPDT_Omron-G5LE-1, F.Cu at (34.5, 77.5)
- added Q1: PN2222A, Package_TO_SOT_THT:TO-92L_Inline_Wide, F.Cu at (37.7, 94.8)
- added R3: 10k, Resistor_THT:R_Axial_DIN0207_L6.3mm_D2.5mm_P10.16mm_Horizontal, F.Cu at (33.5, 91.2)
- added R6: 1k, Resistor_THT:R_Axial_DIN0207_L6.3mm_D2.5mm_P10.16mm_Horizontal, F.Cu at (41.7, 106.9)
- added R7: 1k, Resistor_THT:R_Axial_DIN0207_L6.3mm_D2.5mm_P2.54mm_Vertical, F.Cu at (29.7, 86.0)
- added U2: ESP32-DevKitC, Espressif:ESP32-Nodemcu-india_30pin, F.Cu at (40.5, 143.1)
- D2: footprint LED_THT:LED_D5.0mm_FlatTop -> LED_THT:LED_D3.0mm
- J2: value RELAY -> Screw_Terminal_01x02; footprint Connector_PinHeader_2.54mm:PinHeader_1x04_P2.54mm_Vertical -> TerminalBlock_Phoenix:TerminalBlock_Phoenix_MKDS-1,5-2-5.08_1x02_P5.08mm_Horizontal
- R1: footprint Resistor_THT:R_Axial_DIN0207_L6.3mm_D2.5mm_P2.54mm_Vertical -> Resistor_THT:R_Axial_DIN0204_L3.6mm_D1.6mm_P5.08mm_Horizontal
- moved J2 55.8 mm to (34.1, 51.1), turned to 180 degrees
- moved D3 33.1 mm to (37.3, 121.5), turned to 90 degrees
- moved R4 18.5 mm to (63.5, 72.7), turned to 0 degrees
- moved R5 15.9 mm to (63.5, 76.2), turned to 0 degrees
- moved D2 8.14 mm to (78.8, 123.7), turned to -90 degrees
- moved J4 7.60 mm to (82.1, 114.5)
- moved R2 4.58 mm to (37.2, 104.3), turned to -90 degrees
- moved R1 4.55 mm to (78.8, 134.1)
- moved J3 3.94 mm to (53.4, 48.0)
- moved C2 2.20 mm to (78.8, 136.8)
- moved J1 2.14 mm to (31.2, 135.4)
- moved D1 1.60 mm to (49.4, 141.0)
Connections:
- J2 pad 1: +5V -> Net-(J2-Pin_1)
- J2 pad 2: RLY1 -> Net-(J2-Pin_2)
- J4 pad 4: +3V3 -> +5V
Routing:
- net +12V: track 25.6 -> 129.3 mm
- net Net-(J2-Pin_1): track 0.00 -> 26.6 mm
- net Net-(D4-A): track 0.00 -> 16.7 mm
- net +3V3: track 73.5 -> 60.3 mm, vias 2 -> 0
- net Net-(J2-Pin_2): track 0.00 -> 12.4 mm
- net Net-(Q1-B): track 0.00 -> 12.2 mm
- net RLY2: track 10.8 -> 0.00 mm
- net TX2: track 18.1 -> 10.8 mm
- net RX2: track 18.1 -> 10.8 mm
- net RLY1: track 10.8 -> 4.13 mm
- net +5V: track 179.3 -> 173.1 mm, vias 2 -> 4
- net GND: track 18.9 -> 14.3 mm
- net Net-(D2-A): track 7.20 -> 2.73 mm
- net SCL: track 55.0 -> 59.1 mm
- net Net-(D3-A): track 7.83 -> 4.46 mm
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