File: kicad/iot_power/iot_power.kicad_sch (KiCad schematic)
At the start: 15 parts, among them J1 POWER_SOURCE, J2 RELAY, J3 OLED, J4 PZEM004T, U1 L7805CV

Commit message: nov 25
Parts:
- removed 11: ESP32-DevKitC, Espressif:ESP32-Nodemcu-india, symbol Espressif:ESP32-DevKitC
- removed J2: RELAY, Connector_PinHeader_2.54mm:PinHeader_1x04_P2.54mm_Vertical, symbol Connector_Generic:Conn_01x04
- added D4: 1N4148, Diode_THT:D_DO-35_SOD27_P7.62mm_Horizontal, symbol Diode:1N4148
- added D5: LED, LED_THT:LED_D3.0mm, symbol Device:LED
- added J2: Screw_Terminal_01x02, TerminalBlock_Phoenix:TerminalBlock_Phoenix_MKDS-1,5-2-5.08_1x02_P5.08mm_Horizontal, symbol Connector:Screw_Terminal_01x02
- added K1: G5LE-1, Relay_THT:Relay_SPDT_Omron-G5LE-1, symbol Relay:G5LE-1
- added Q1: PN2222A, Package_TO_SOT_THT:TO-92L_Inline_Wide, symbol Transistor_BJT:PN2222A
- added R3: 10k, Resistor_THT:R_Axial_DIN0207_L6.3mm_D2.5mm_P10.16mm_Horizontal, symbol Device:R_US
- added R6: 1k, Resistor_THT:R_Axial_DIN0207_L6.3mm_D2.5mm_P10.16mm_Horizontal, symbol Device:R_US
- added R7: 1k, Resistor_THT:R_Axial_DIN0207_L6.3mm_D2.5mm_P2.54mm_Vertical, symbol Device:R_US
- added U2: ESP32-DevKitC, Espressif:ESP32-Nodemcu-india_30pin, symbol Espressif:ESP32-india-30Pin
- D2: footprint LED_THT:LED_D5.0mm_FlatTop -> LED_THT:LED_D3.0mm
- R1: footprint Resistor_THT:R_Axial_DIN0207_L6.3mm_D2.5mm_P2.54mm_Vertical -> Resistor_THT:R_Axial_DIN0204_L3.6mm_D1.6mm_P5.08mm_Horizontal
Connections:
- net +12V: now also D4.1 (K), K1.5, R7.1
- net +3V3: now also U2.16 (3V3); no longer J4.4 (Pin_4)
- net +5V: now also J4.4 (Pin_4), U2.15 (VIN)
- net CLED: now also U2.8 (DAC_1/ADC2_CH8/GPIO25)
- net GND: now also Q1.1 (E), R3.2, U2.14 (GND), U2.17 (GND)
- net RLY1: now also R6.1, U2.9 (DAC_2/ADC2_CH9/GPIO26)
- net RX2: now also U2.21 (RX2/GPIO16)
- net SCL: now also U2.29 (GPIO22/SCL)
- net SDA: now also U2.26 (GPIO21/SDA)
- net TX2: now also U2.22 (TX2/GPIO17)
- new net: Q1.2 (B), R3.1, R6.2
- new net: D5.2 (A), R7.2
- new net: J2.1 (Pin_1), K1.1
- new net: D4.2 (A), D5.1 (K), K1.2, Q1.3 (C)
- new net: J2.2 (Pin_2), K1.4
